File: battery switch delay.kicad_sch (KiCad schematic)
At the start: 11 parts, among them J1 5mm pitch 4 position screw te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, K2 G6E-134P-US, Q1 2N3904, U2 MIC2920A-12WS-TR_SOT223

Commit message: got the transistor the correct footprint hopefully
Parts:
- removed Q1: 2N3904, Package_TO_SOT_THT:TO-92_Inline, symbol Transistor_BJT:2N3904
- added Q1: Q_NPN, Package_TO_SOT_SMD:SOT-23, symbol Device:Q_NPN
Connections:
- net GND: now also Q1.2 (E)
- net at K2.12, R1.2: now also Q1.3 (C)
- net at R3.1: now also Q1.1 (B)
Changed lines of the file:
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@@
+	)
+	(symbol
+		(lib_id "Device:Q_NPN")
+		(at 60.96 111.76 0)
+		(mirror y)
+		(unit 1)
+		(exclude_from_sim no)
+		(in_bom yes)
+		(on_board yes)
+		(dnp no)
+		(property "Reference" "Q1"
+			(at 55.88 110.4899 0)
+			(effects
+				(font
+					(size 1.27 1.27)
+				)
+				(justify left)
+			)
+		)
+		(property "Value" "Q_NPN"
+			(at 55.88 113.0299 0)
+			(effects
+				(font
+					(size 1.27 1.27)
+				)
+				(justify left)
+			)
+		)
+		(property "Footprint" "Package_TO_SOT_SMD:SOT-23"
+			(at 55.88 109.22 0)
+			(effects
+				(font
+					(size 1.27 1.27)
+				)
+				(hide yes)
+			)
+		)
+		(property "Datasheet" "~"
+			(at 60.96 111.76 0)
+			(effects
+				(font
+					(size 1.27 1.27)
+				)
+				(hide yes)
+			)
+		)
+		(property "Description" "NPN bipolar junction transistor"
+			(at 60.96 111.76 0)
+			(effects
+				(font
+					(size 1.27 1.27)
+				)
+				(hide yes)
+			)
+		)
+		(pin "3"
+		)
+		(pin "1"
+		)
+		(pin "2"
+		)
+		(instances
+			(project ""
+				(path "/72486ea4-2971-4ca2-ab8b-187d20cf76b7"
+					(reference "Q1")
+					(unit 1)
+				)
+			)
+		)
 	)
 	(symbol
@@
 					(unit 1)
 				)
-			)
-		)
-	)
-	(symbol
-		(lib_id "Transistor_BJT:2N3904")
-		(at 60.96 111.76 0)
-		(mirror y)
-		(unit 1)
-		(exclude_from_sim no)
-		(in_bom yes)
-		(on_board yes)
-		(dnp no)
-		(property "Reference" "Q1"
-			(at 55.88 110.4899 0)
-			(effects
-				(font
-					(size 1.27 1.27)
-				)
-				(justify left)
-			)
-		)
-		(property "Value" "2N3904"
-			(at 55.88 113.0299 0)
-			(effects
-				(font
-					(size 1.27 1.27)
-				)
-				(justify left)
-			)
-		)
-		(property "Footprint" "Package_TO_SOT_THT:TO-92_Inline"
-			(at 55.88 113.665 0)
-			(effects
-				(font
-					(size 1.27 1.27)
-					(italic yes)
-				)
-				(justify left)
-				(hide yes)
-			)
-		)
-		(property "Datasheet" "https://www.onsemi.com/pub/Collateral/2N3903-D.PDF"
-			(at 60.96 111.76 0)
-			(effects
-				(font
-					(size 1.27 1.27)
-				)
-				(justify left)
-				(hide yes)
-			)
-		)
-		(property "Description" "0.2A Ic, 40V Vce, Small Signal NPN Transistor, TO-92"
-			(at 60.96 111.76 0)
-			(effects
-				(font
-					(size 1.27 1.27)
-				)
-				(hide yes)
-			)
-		)
-		(pin "3"
-		)
-		(pin "2"
-		)
-		(pin "1"
-		)
-		(instances
-			(project ""
-				(path "/72486ea4-2971-4ca2-ab8b-187d20cf76b7"
-					(reference "Q1")
-					(unit 1)
-				)

Commit message: did more board layout and actualy have all nets connected. looking at drc so i can be sure
Changed lines of the file:
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@@
 	(wire
 		(pts
-			(xy 17.78 66.04) (xy 38.1 66.04)
+			(xy 20.32 66.04) (xy 38.1 66.04)
 		)
 		(stroke
@@
 	(wire
 		(pts
-			(xy 17.78 66.04) (xy 17.78 82.55)
+			(xy 20.32 66.04) (xy 20.32 69.85)
 		)
 		(stroke
@@
 			)
 		)
-		(property "Description" "500mW Zener Diode, DO-35"
+		(property "Description" "Zener Diode"
 			(at 90.17 88.9 0)
 			(effects
@@
 	(symbol
 		(lib_id "power:+12V")
-		(at 17.78 82.55 180)
+		(at 20.32 69.85 180)
 		(unit 1)
 		(exclude_from_sim no)
@@
 		(dnp no)
 		(property "Reference" "#PWR09"
-			(at 17.78 78.74 0)
+			(at 20.32 66.04 0)
 			(effects
 				(font
@@
 		)
 		(property "Value" "to switch"
-			(at 17.78 87.63 0)
+			(at 20.32 74.93 0)
 			(effects
 				(font
@@
 		)
 		(property "Footprint" ""
-			(at 17.78 82.55 0)
+			(at 20.32 69.85 0)
 			(effects
 				(font
@@
 		)
 		(property "Datasheet" ""
-			(at 17.78 82.55 0)
+			(at 20.32 69.85 0)
 			(effects
 				(font
@@
 		)
 		(property "Description" "Power symbol creates a global label with name \"+12V\""
-			(at 17.78 82.55 0)
-			(effects
-				(font
+			(at 20.32 69.85 0)
+			(effects
+				(font
